Commit message: update ws

File: src/pmzbbot_description/description/pmzbbot_core.urdf.xacro (robot description, xacro)
@@ -36,13 +36,8 @@
         <link name="chassis">
         <visual>
-            <!-- <origin xyz="${chassis_length/2} 0 ${chassis_height/2}"/> -->
-            <origin xyz="${chassis_length/2} 0 -0.10"/>
-            <!-- <geometry>
+            <origin xyz="${chassis_length/2} 0 ${chassis_height/2}"/>
+            <geometry>
                 <box size="${chassis_length} ${chassis_width} ${chassis_height}"/>
-            </geometry> -->
-            <geometry>
-                <mesh filename="file://$(find zhbbot_description)/meshes/mir_100_base.stl"/>
-            </geometry>
-            <material name="grey"/>
+            </geometry>
         </visual>
         <collision>
