Commit message: Update Robot Description

File: src/pmzbbot_description/description/pmzbbot.urdf.xacro (robot description, xacro)
@@ -2,4 +2,4 @@
 <robot xmlns:xacro="http://www.ros.org/wiki/xacro"  name="robot">
     <xacro:include filename="pmzbbot_core.urdf.xacro" />
-    <xacro:zhbbot_core/>
+    <xacro:pmzbbot_core/>
 </robot>

File: src/pmzbbot_description/description/pmzbbot_common.xacro (robot description, xacro)
@@ -33,5 +33,5 @@
     </inertial>
     </xacro:macro>
-  <xacro:macro name="zhbbot_common">
+  <xacro:macro name="pmzbbot_common">
     <!-- Mobile Robot Parameter -->
     <xacro:property name="wheel_radius" value="0.034" scope="parent"/>
@@ -39,8 +39,13 @@
     <xacro:property name="wheel_mass" value="0.029" scope="parent"/>
     <xacro:property name="wheel_offset_y" value="0.0805" scope="parent"/>
+    <xacro:property name="casterwheel_mass" value="0.042" scope="parent"/>
+    <xacro:property name="casterwheel_radius" value="0.018" scope="parent"/>
+    <xacro:property name="casterwheel_offset_x" value="0.097" scope="parent"/>
+    <xacro:property name="casterwheel_offset_z" value="0.016" scope="parent"/>
     <xacro:property name="chassis_length" value="0.15" scope="parent"/>
-    <xacro:property name="chassis_width" value="0.161" scope="parent"/>
+    <xacro:property name="chassis_width" value="0.136" scope="parent"/>
     <xacro:property name="chassis_height" value="0.0915" scope="parent"/>
     <xacro:property name="chassis_offset_x" value="0.027" scope="parent"/>
+    <xacro:property name="chassis_offset_z" value="0.016" scope="parent"/>
     <xacro:property name="battery_mass" value="0.207" scope="parent"/>
     <xacro:property name="leftmotor_mass" value="0.057" scope="parent"/>
@@ -49,7 +54,7 @@
     <xacro:property name="imu_mass" value="0.040" scope="parent"/>
     <xacro:property name="base_mass" value="0.094" scope="parent"/>
-    <xacro:property name="casterwheel_mass" value="0.055" scope="parent"/>
     <xacro:property name="other_mass" value="0.055" scope="parent"/>
-    <xacro:property name="chassis_mass" value="${battery_mass + leftmotor_mass + rightmotor_mass + esp32_mass + imu_mass + base_mass + casterwheel_mass + other_mass}" scope="parent"/>
+    <xacro:property name="caster3d_mass" value="0.012" scope="parent"/>
+    <xacro:property name="chassis_mass" value="${battery_mass + leftmotor_mass + rightmotor_mass + esp32_mass + imu_mass + base_mass + other_mass + caster3d_mass}" scope="parent"/>
   </xacro:macro>
 </robot>

File: src/pmzbbot_description/description/pmzbbot_core.urdf.xacro (robot description, xacro)
@@ -4,9 +4,9 @@
         <xacro:include filename="inertial_macros.xacro" />
         <xacro:include filename="pmzbbot_common.xacro" />
-        <xacro:zhbbot_common/>
+        <xacro:pmzbbot_common/>
         <xacro:include filename="pmzbbot_ros2control.xacro" />
-        <xacro:zhbbot_control/>
-        <!-- BASE_FOOTPRINT LINK -->
-        <link name="base_footprint">
+        <xacro:pmzbbot_control/>
+        <!-- BASE LINK -->
+        <link name="base_link">
         </link>
         <!-- For Velocity Controller -->
@@ -16,25 +16,19 @@
             <origin xyz="0 0 -${wheel_radius}" rpy="0 0 0"/>
         </joint>
-        <!-- For Differantial Drive Controller -->
-        <!-- <joint name="base_footprint_joint" type="fixed">
-            <parent link="base_link"/>
-            <child link="base_footprint"/>
-            <origin xyz="0 0 0" rpy="0 0 0"/>
-        </joint> -->
+        <!-- BASE_FOOTPRINT LINK -->
+        <link name="base_footprint">
+        </link>
         <!-- <origin xyz="0 0 ${-wheel_radius + wheel_offset_z}" rpy="0 0 0"/> -->
-        <!-- BASE LINK -->
-        <link name="base_link">
-        </link>
         <!-- CHASSIS Information -->
         <!--joint-->
         <joint name="chassis_joint" type="fixed">
-        <parent link="base_link"/>
-        <child link="chassis"/>
-        <origin xyz="${-wheel_offset_x} 0 ${-wheel_offset_z}"/>
+            <parent link="base_link"/>
+            <child link="chassis_link"/>
+            <origin xyz="${-chassis_offset_x} 0 0"/>
         </joint>
         <!--link-->
-        <link name="chassis">
+        <link name="chassis_link">
         <visual>
-            <origin xyz="${chassis_length/2} 0 ${chassis_height/2}"/>
+            <origin xyz="${chassis_length/2} 0 ${(chassis_height/2 - chassis_offset_z)}"/>
             <geometry>
                 <box size="${chassis_length} ${chassis_width} ${chassis_height}"/>
@@ -42,15 +36,11 @@
         </visual>
         <collision>
-            <!-- <origin xyz="${chassis_length/2} 0 ${chassis_height/2}"/> -->
-            <origin xyz="${chassis_length/2} 0 -0.10"/>
-            <!-- <geometry>
+            <origin xyz="${chassis_length/2} 0 ${(chassis_height/2 - chassis_offset_z)}"/>
+            <geometry>
                 <box size="${chassis_length} ${chassis_width} ${chassis_height}"/>
-            </geometry> -->
-            <geometry>
-                <mesh filename="file://$(find zhbbot_description)/meshes/mir_100_base.stl"/>
             </geometry>
         </collision>
-        <xacro:inertial_box mass="100" x="${chassis_length}" y="${chassis_width}" z="${chassis_height}">
-            <origin xyz="${chassis_length/2} 0 ${chassis_height/2}" rpy="0 0 0"/>
+        <xacro:inertial_box mass="${chassis_mass}" x="${chassis_length}" y="${chassis_width}" z="${chassis_height}">
+            <origin xyz="${chassis_length/2} 0 ${(chassis_height/2)}" rpy="0 0 0"/>
         </xacro:inertial_box>
         </link>
@@ -108,13 +98,13 @@
         </gazebo>
         <!-- CASTER WHEEL FONT RIGHT -->
-        <joint name="caster_wheel_f_r_joint" type="fixed">
+        <joint name="caster_wheel_joint" type="fixed">
             <parent link="base_link"/>
-            <child link="caster_wheel_f_r"/>
-            <origin xyz="${caster_wheel_offset_x} ${caster_wheel_offset_y} ${caster_wheel_offset_z}"/>
+            <child link="caster_wheel"/>
+            <origin xyz="${casterwheel_offset_x} 0 -${casterwheel_offset_z}"/>
         </joint>
-        <link name="caster_wheel_f_r">
+        <link name="caster_wheel">
             <visual>
                 <geometry>
-                    <sphere radius="${caster_wheel_radius}"/>
+                    <sphere radius="${casterwheel_radius}"/>
                 </geometry>
                 <material name="white"/>
@@ -122,147 +112,15 @@
             <collision>
                 <geometry>
-                    <sphere radius="${caster_wheel_radius}"/>
+                    <sphere radius="${casterwheel_radius}"/>
                 </geometry>
             </collision>
-            <xacro:inertial_sphere mass="${caster_wheel_mass}" radius="${caster_wheel_radius}">
+            <xacro:inertial_sphere mass="${casterwheel_mass}" radius="${casterwheel_radius}">
                 <origin xyz="0 0 0" rpy="0 0 0"/>
             </xacro:inertial_sphere>
         </link>
-        <gazebo reference="caster_wheel_f_r">
+        <gazebo reference="caster_wheel">
             <material>Gazebo/Blue</material>
             <mu1 value="0.001"/>
             <mu2 value="0.001"/>
-        </gazebo>
-        <!-- CASTER WHEEL FONT LEFT -->
-        <joint name="caster_wheel_f_l_joint" type="fixed">
-            <parent link="base_link"/>
-            <child link="caster_wheel_f_l"/>
-            <origin xyz="${caster_wheel_offset_x} ${-caster_wheel_offset_y} ${caster_wheel_offset_z}"/>
-        </joint>
-        <link name="caster_wheel_f_l">
-            <visual>
-                <geometry>
-                    <sphere radius="${caster_wheel_radius}"/>
-                </geometry>
-                <material name="white"/>
-            </visual>
-            <collision>
-                <geometry>
-                    <sphere radius="${caster_wheel_radius}"/>
-                </geometry>
-            </collision>
-            <xacro:inertial_sphere mass="${caster_wheel_mass}" radius="${caster_wheel_radius}">
-                <origin xyz="0 0 0" rpy="0 0 0"/>
-            </xacro:inertial_sphere>
-        </link>
-        <gazebo reference="caster_wheel_f_l">
-            <material>Gazebo/Blue</material>
-            <mu1 value="0.001"/>
-            <mu2 value="0.001"/>
-        </gazebo>
-        <!-- CASTER WHEEL BACK RIGHT -->
-        <joint name="caster_wheel_r_r_joint" type="fixed">
-            <parent link="base_link"/>
-            <child link="caster_wheel_r_r"/>
-            <origin xyz="${-caster_wheel_offset_x} ${caster_wheel_offset_y} ${caster_wheel_offset_z}"/>
-        </joint>
-        <link name="caster_wheel_r_r">
-            <visual>
-                <geometry>
-                    <sphere radius="${caster_wheel_radius}"/>
-                </geometry>
-                <material name="white"/>
-            </visual>
-            <collision>
-                <geometry>
-                    <sphere radius="${caster_wheel_radius}"/>
-                </geometry>
-            </collision>
-            <xacro:inertial_sphere mass="${caster_wheel_mass}" radius="${caster_wheel_radius}">
-                <origin xyz="0 0 0" rpy="0 0 0"/>
-            </xacro:inertial_sphere>
-        </link>
-        <gazebo reference="caster_wheel_r_r">
-            <material>Gazebo/Blue</material>
-            <mu1 value="0.001"/>
-            <mu2 value="0.001"/>
-        </gazebo>
-        <!-- CASTER WHEEL BACK LEFT -->
-        <joint name="caster_wheel_r_l_joint" type="fixed">
-            <parent link="base_link"/>
-            <child link="caster_wheel_r_l"/>
-            <origin xyz="${-caster_wheel_offset_x} ${-caster_wheel_offset_y} ${caster_wheel_offset_z}"/>
-        </joint>
-        <link name="caster_wheel_r_l">
-            <visual>
-                <geometry>
-                    <sphere radius="${caster_wheel_radius}"/>
-                </geometry>
-                <material name="white"/>
-            </visual>
-            <collision>
-                <geometry>
-                    <sphere radius="${caster_wheel_radius}"/>
-                </geometry>
-            </collision>
-            <xacro:inertial_sphere mass="${caster_wheel_mass}" radius="${caster_wheel_radius}">
-                <origin xyz="0 0 0" rpy="0 0 0"/>
-            </xacro:inertial_sphere>
-        </link>
-        <gazebo reference="caster_wheel_r_l">
-            <material>Gazebo/Black</material>
-            <mu1 value="0.001"/>
-            <mu2 value="0.001"/>
-        </gazebo>
-        <!-- Laser  -->
-        <joint name="laser_joint" type="fixed">
-            <parent link="base_link"/>
-            <child link="lidar_link"/>
-            <origin xyz="0.122 0 0.312" rpy="0 0 0"/>
-        </joint>
-        <link name="lidar_link">
-            <visual>
-                <geometry>
-                    <cylinder radius="0.05" length="0.04"/>
-                </geometry>
-                <material name="red"/>
-            </visual>
-            <visual>
-                <origin xyz="0 0 -0.05"/>
-                <geometry>
-                    <cylinder radius="0.01" length="0.1"/>
-                </geometry>
-                <material name="red"/>
-            </visual>
-        </link>
-        <gazebo reference="lidar_link">
-                <material>Gazebo/Red</material>
-        </gazebo>
-        <gazebo reference="lidar_link">
-            <sensor name="laser" type="ray">
-                <pose> 0 0 0 0 0 0 </pose>
-                <visualize>true</visualize>
-                <update_rate>5</update_rate>
-                <ray>
-                    <scan>
-                        <horizontal>
-                            <samples>360</samples>
-                            <min_angle>-3.14</min_angle>
-                            <max_angle>3.14</max_angle>
-                        </horizontal>
-                    </scan>
-                    <range>
-                        <min>0.25</min>
-                        <max>20</max>
-                    </range>
-                </ray>
-                <plugin name="laser_controller" filename="libgazebo_ros_ray_sensor.so">
-                    <ros>
-                        <argument>~/out:=scan</argument>
-                    </ros>
-                    <output_type>sensor_msgs/LaserScan</output_type>
-                    <frame_name>lidar_link</frame_name>
-                </plugin>
-            </sensor>
         </gazebo>
         <!-- Ground truth pose -->
