Commit message: clean project

File: src/pmzbbot_description/description/pmzbbot_common.xacro (robot description, xacro)
@@ -24,13 +24,4 @@
         <color rgba="0.0 0.0 0.3764 0.6"/>
     </material>
-    <xacro:macro name="cylinder_inertial" params="radius length mass *origin">
-    <inertial>
-      <mass value="${mass}" />
-      <xacro:insert_block name="origin" />
-      <inertia ixx="${0.0833333 * mass * (3 * radius * radius + length * length)}" ixy="0.0" ixz="0.0"
-        iyy="${0.0833333 * mass * (3 * radius * radius + length * length)}" iyz="0.0"
-        izz="${0.5 * mass * radius * radius}" />
-    </inertial>
-    </xacro:macro>
   <xacro:macro name="pmzbbot_common">
     <!-- Mobile Robot Parameter -->

File: src/pmzbbot_description/description/pmzbbot_core.urdf.xacro (robot description, xacro)
@@ -5,6 +5,4 @@
         <xacro:include filename="pmzbbot_common.xacro" />
         <xacro:pmzbbot_common/>
-        <xacro:include filename="pmzbbot_ros2control.xacro" />
-        <xacro:pmzbbot_control/>
         <!-- BASE LINK -->
         <link name="base_link">
